File: simulations/lab1/kicad/lab1-exp4-bridge-rc.kicad_sch (KiCad schematic)
At the start: 6 parts

Commit message: fix: 實驗四的二極體編號與講義不符，且虛線原語在短線段上被畫成實線
- **修正** 實驗四三張電流分析圖與筆記內文、表格一律改用講義編號：正半週 D3、D1，負半週 D4、D2（原本寫成 D2、D4 與 D1、D3）；四顆二極體旁另加 D1–D4 標籤。已比對講義 PDF p22／p25 的電路圖符號方向確認
- **修正** `current_overlay.py` 的虛線改成沿線長等距切段。原本把整段均分成 n 份，麵包板上的短線段只切得出一兩格、缺口又被中點的箭頭蓋住，整段看起來就是實線
- **修正** KiCad `lab1-exp4-bridge` 圖上註記的電流路徑 D1／D2 對調（符號本身是對的），並重新匯出 svg／sheet／pdf
- **修正** 實驗三負半週與放電圖中沒有電流的線段改為細虛線且不畫方向箭頭
- **修正** 實驗三放電圖的結論：半波兩個峰值之間要撐將近一整個週期（16.7 ms）而非半週期，輸出會從約 4.3 V 掉到約 1.3 V
- **修正** 九處編號位置與步驟文字對不上的問題（例如文字寫「第 9 欄的紅跳線」、編號卻擺在第 14 欄），並把編號移出麵包板的欄位號碼
- **修正** 實驗二原理圖 alt text 的二極體方向，以及負半週圖殘留的「箭頭全部反向」描述
- **新增** 實驗三負半週圖的 ①–⑧ 編號，與筆記中正負半週共用的 8 列逐步說明表
- **新增** 第 26 頁「橋式 + 1 µF」小節：Tinkercad 接線圖與充電、放電兩張電流分析圖；底圖裁切與縮放刻意對齊既有座標系，既有路徑常數可直接沿用
- **新增** KiCad `lab1-exp4-bridge-rc` 結報電路圖與產生器 `gen_exp4_rc.py`
- **調整** 齊納段落改寫為「這正是講義要量的 Vin < VZ 情況」，不再斷言講義參數不自洽
- **調整** 補上講義投影片印刷頁碼與 PDF 頁序的對照表，並在實驗四三處雙標
- **調整** Tinkercad 設計總表加入第 26 頁那一版的連結，並更正共用狀態的說明

Co-Authored-By: Claude Opus 5 (1M context) <noreply@anthropic.com>
Claude-Session: https://claude.ai/code/session_01BApRtS8HBwJgXmVwru8eqw
Parts:
- added C1: 1µF, symbol Device:C
Connections:
- net GND: now also C1.2
- net at D3.1 (K), D4.1 (K), RL.1: now also C1.1
Other:
- note added: "C1 與 R_{L} 並聯：Vin 高於電容電壓時充電，低於時由電容單獨供應負載"
- note added: "Lab 1 實驗四（第 26 頁）：全波橋式整流器 + 1 µF 濾波電容"
- note removed: "Lab 1 實驗四：全波橋式整流器量測電路"
- note removed: "第 26 頁在 R_{L} 兩端並聯 C 1 µF；第 27 頁改並聯齊納，陰極朝 P（輸出 +）那側"
- title: Lab 1 實驗四：全波橋式整流器 -> Lab 1 實驗四：全波橋式整流器 + RC 濾波

Commit message: feat(kicad): 五張 Lab 1 原理圖加入 ngspice 模擬指令，可在 KiCad 內建模擬器直接跑
- **新增** `gen_exp1`～`gen_exp4_rc` 各放一行 `.dc`／`.tran` 指令文字，重新產生原理圖、SPICE 網表、SVG 與 PDF，ERC 仍為 0 錯誤
- **調整** `kicad/README.md` 說明 GUI 模擬步驟與 `kicad-cli` 沒有 `sim` 子命令的限制
- **調整** 筆記用的 `public/note-images/ec-week3-kicad/` 五張圖同步

Co-Authored-By: Claude Fable 5.1 <noreply@anthropic.com>
Claude-Session: https://claude.ai/code/session_01CSTJPweMCqSNGPRV9i9S1L
Other:
- note added: ".tran 10u 200m"
